File: PCBs/Rotary Switches/Rotary Switches.kicad_sch (KiCad schematic)
At the start: 8 parts, among them J1 Conn_01x03_Pin, SW1 A12505RNCQ

Commit message: Release Rotary Switch PCB version 1.2 with ON/OFF solder jumper
Parts:
- added JP1: ON/OFF, Jumper:SolderJumper-2_P1.3mm_Open_Pad1.0x1.5mm, symbol Jumper:SolderJumper_2_Open
Connections:
- net GND: now also JP1.2 (B)
- net TAP_1: now also JP1.1 (A)
Other:
- note added: "ON/OFF option: omit R1-R6, bridge JP1. J1 pin 2 to Teensy input with pull-up. Ladder option: fit R1-R6 and leave JP1 open."
Changed lines of the file:
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@@
 	(generator_version "10.0")
 	(paper "A")
+	(text "ON/OFF option: omit R1-R6, bridge JP1. J1 pin 2 to Teensy input with pull-up.\nLadder option: fit R1-R6 and leave JP1 open."
+		(exclude_from_sim no)
+		(at 71.12 153.67 0)
+		(effects
+			(font
+				(size 1.27 1.27)
+			)
+		)
+	)
 	(text "J1: 1 = 3.3V, 2 = analog output, 3 = GND\nSix 1k resistors provide seven ladder voltages; terminal 11 is unused."
 		(exclude_from_sim no)
@@
 	(label "TAP_3"
 		(at 69.85 102.87 90)
+		(effects
+			(font
+				(size 1 1)
+			)
+			(justify left bottom)
+		)
+	)
+	(label "TAP_1"
+		(at 66.04 142.24 0)
+		(effects
+			(font
+				(size 1 1)
+			)
+			(justify left bottom)
+		)
+	)
+	(label "GND"
+		(at 76.2 142.24 0)
 		(effects
 			(font
@@
 					(unit 1)
 				)
+			)
+		)
+	)
+	(symbol
+		(lib_id "Jumper:SolderJumper_2_Open")
+		(at 71.12 142.24 0)
+		(unit 1)
+		(body_style 1)
+		(exclude_from_sim no)
+		(in_bom no)
+		(on_board yes)
+		(in_pos_files yes)
+		(dnp no)
+		(property "Reference" "JP1"
+			(at 71.12 138.43 0)
+			(show_name no)
+			(do_not_autoplace no)
+			(effects
+				(font
+					(size 1.27 1.27)
+				)
+			)
+		)
+		(property "Value" "ON/OFF"
+			(at 71.12 146.05 0)
+			(show_name no)
+			(do_not_autoplace no)
+			(effects
+				(font
+					(size 1.27 1.27)
+				)
+			)
+		)
+		(property "Footprint" "Jumper:SolderJumper-2_P1.3mm_Open_Pad1.0x1.5mm"
+			(at 71.12 142.24 0)
+			(hide yes)
+			(show_name no)
+			(do_not_autoplace no)
+			(effects
+				(font
+					(size 1.27 1.27)
+				)
+			)
+		)
+		(property "Datasheet" ""
+			(at 71.12 142.24 0)
+			(show_name no)
+			(do_not_autoplace no)
+			(effects
+				(font
+					(size 1.27 1.27)
+				)
+			)
+		)
+		(property "Description" ""
+			(at 71.12 142.24 0)
+			(show_name no)
+			(do_not_autoplace no)
+			(effects
+				(font
+					(size 1.27 1.27)
+				)
+			)
+		)
+		(pin "1"
+		)
+		(pin "2"
+		)
+		(instances
+			(project "Rotary Switches"
+				(path "/b968bbd6-d719-4aab-adf0-78b0284df4a7"
+					(reference "JP1")
+					(unit 1)
+				)
