File: PCBs/Rotary Encoders/Rotary Encoders.kicad_pcb (KiCad board)
At the start: 2 copper layers, 45.7 x 108.8 mm, 7 parts, among them J1 Conn_01x14_Pin, SW1 RotaryEncoder_Switch, SW2 RotaryEncoder_Switch, SW3 RotaryEncoder_Switch, SW4 RotaryEncoder_Switch, SW5 RotaryEncoder_Switch, SW6 RotaryEncoder_Switch

Commit message: Publish Rotary Encoder PCB v1.1 with corrected power GND connections
Other:
- board text added: "ARC-210 Rotary Encoder v1.1"
- board text removed: "ARC-210 Rotary Encoder v1.0"
Changed lines of the file:
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@@
 		)
 		(embedded_fonts no)
-		(model "${KIPRJMOD}/PEC11H-4220F-S0024.stp"
+		(model "PEC11H-4220F-S0024.stp"
 			(offset
 				(xyz 2.499999962 7.489999659 2.229999986)
@@
 		)
 		(embedded_fonts no)
-		(model "${KIPRJMOD}/PEC11H-4220F-S0024.stp"
+		(model "PEC11H-4220F-S0024.stp"
 			(offset
 				(xyz 2.499999962 7.489999659 2.229999986)
@@
 		)
 		(embedded_fonts no)
-		(model "${KIPRJMOD}/PEC11H-4220F-S0024.stp"
+		(model "PEC11H-4220F-S0024.stp"
 			(offset
 				(xyz 2.499999962 7.489999659 2.229999986)
@@
 		)
 		(embedded_fonts no)
-		(model "${KIPRJMOD}/PEC11H-4220F-S0024.stp"
+		(model "PEC11H-4220F-S0024.stp"
 			(offset
 				(xyz 2.499999962 7.489999659 2.229999986)
@@
 		)
 		(embedded_fonts no)
-		(model "${KIPRJMOD}/PEC11H-4220F-S0024.stp"
+		(model "PEC11H-4220F-S0024.stp"
 			(offset
 				(xyz 2.499999962 7.489999659 2.229999986)
@@
 		)
 	)
-	(gr_text "ARC-210 Rotary Encoder v1.0"
+	(gr_text "ARC-210 Rotary Encoder v1.1"
 		(at 105.6 89.3 90)
 		(layer "B.SilkS")
@@
 	)
 	(segment
+		(start 120 95)
+		(end 120.083719 95)
+		(width 0.2)
+		(layer "F.Cu")
+		(net "Net-(J1-Pin_13)")
+	)
+	(segment
+		(start 126.895 94.275)
+		(end 125.825 95.345)
+		(width 0.2)
+		(layer "F.Cu")
+		(net "Net-(J1-Pin_13)")
+	)
+	(segment
+		(start 115 90)
+		(end 120 95)
+		(width 0.2)
+		(layer "F.Cu")
+		(net "Net-(J1-Pin_13)")
+	)
+	(segment
+		(start 138.25 90)
+		(end 133.975 94.275)
+		(width 0.2)
+		(layer "F.Cu")
+		(net "Net-(J1-Pin_13)")
+	)
+	(segment
+		(start 120.083719 95)
+		(end 120.427091 95.343372)
+		(width 0.2)
+		(layer "F.Cu")
+		(net "Net-(J1-Pin_13)")
+	)
+	(segment
+		(start 133.975 94.275)
+		(end 126.895 94.275)
+		(width 0.2)
+		(layer "F.Cu")
+		(net "Net-(J1-Pin_13)")
+	)
+	(segment
+		(start 113.775 82.15)
+		(end 115.05 83.425)
+		(width 0.2)
+		(layer "F.Cu")
+		(net "Net-(J1-Pin_13)")
+	)
+	(segment
+		(start 113.775 81.55)
+		(end 113.775 82.15)
+		(width 0.2)
+		(layer "F.Cu")
+		(net "Net-(J1-Pin_13)")
+	)
+	(via
+		(at 120.427091 95.343372)
+		(size 0.6)
+		(drill 0.3)
+		(layers "F.Cu" "B.Cu")
+		(net "Net-(J1-Pin_13)")
+	)
+	(via
+		(at 113.775 81.55)
+		(size 0.6)
+		(drill 0.3)
+		(layers "F.Cu" "B.Cu")
+		(net "Net-(J1-Pin_13)")
+	)
+	(via
+		(at 115.05 83.425)
+		(size 0.6)
+		(drill 0.3)
+		(layers "F.Cu" "B.Cu")
+		(net "Net-(J1-Pin_13)")
+	)
+	(segment
+		(start 125.825 95.345)
+		(end 124.855 95.345)
+		(width 0.2)
+		(layer "B.Cu")
+		(net "Net-(J1-Pin_13)")
+	)
+	(segment
+		(start 123.283372 95.343372)
+		(end 124.07 96.13)
+		(width 0.2)
+		(layer "B.Cu")
+		(net "Net-(J1-Pin_13)")
+	)
+	(segment
+		(start 111.95 78.175)
+		(end 111.95 79.725)
+		(width 0.2)
+		(layer "B.Cu")
+		(net "Net-(J1-Pin_13)")
+	)
+	(segment
+		(start 115 75.125)
+		(end 111.95 78.175)
+		(width 0.2)
+		(layer "B.Cu")
+		(net "Net-(J1-Pin_13)")
+	)
+	(segment
+		(start 124.07 96.13)
+		(end 125.825 97.885)
+		(width 0.2)
+		(layer "B.Cu")
+		(net "Net-(J1-Pin_13)")
+	)
+	(segment
+		(start 125.825 115.825)
+		(end 125.825 97.885)
+		(width 0.2)
+		(layer "B.Cu")
+		(net "Net-(J1-Pin_13)")
+	)
+	(segment
+		(start 115.05 83.425)
+		(end 115 83.475)
+		(width 0.2)
+		(layer "B.Cu")
+		(net "Net-(J1-Pin_13)")
+	)
+	(segment
+		(start 115 111.5)
+		(end 119.45 115.95)
+		(width 0.2)
+		(layer "B.Cu")
+		(net "Net-(J1-Pin_13)")
+	)
+	(segment
+		(start 111.95 79.725)
+		(end 113.775 81.55)
+		(width 0.2)
+		(layer "B.Cu")
+		(net "Net-(J1-Pin_13)")
+	)
+	(segment
+		(start 120.427091 95.343372)
+		(end 123.283372 95.343372)
+		(width 0.2)
+		(layer "B.Cu")
+		(net "Net-(J1-Pin_13)")
+	)
+	(segment
+		(start 115 47)
+		(end 115 68.5)
+		(width 0.2)
+		(layer "B.Cu")
+		(net "Net-(J1-Pin_13)")
+	)
+	(segment
+		(start 115 68.5)
+		(end 115 75.125)
+		(width 0.2)
+		(layer "B.Cu")
+		(net "Net-(J1-Pin_13)")
+	)
+	(segment
+		(start 115 133)
+		(end 115 111.5)
+		(width 0.2)
+		(layer "B.Cu")
+		(net "Net-(J1-Pin_13)")
+	)
+	(segment
+		(start 119.45 115.95)
+		(end 125.95 115.95)
+		(width 0.2)
+		(layer "B.Cu")
+		(net "Net-(J1-Pin_13)")
+	)
+	(segment
+		(start 124.855 95.345)
+		(end 124.07 96.13)
+		(width 0.2)
+		(layer "B.Cu")
+		(net "Net-(J1-Pin_13)")
+	)
+	(segment
+		(start 125.95 115.95)
+		(end 125.825 115.825)
+		(width 0.2)
+		(layer "B.Cu")
+		(net "Net-(J1-Pin_13)")
+	)
+	(segment
+		(start 115 83.475)
+		(end 115 90)
+		(width 0.2)
+		(layer "B.Cu")
+		(net "Net-(J1-Pin_13)")
+	)
+	(segment
 		(start 120.7 103.01)
 		(end 120.7 104)
@@
 		(net "Net-(J1-Pin_8)")
 	)
-	(segment
-		(start 120 95)
-		(end 120.083719 95)
-		(width 0.2)
-		(layer "F.Cu")
-		(net "Net-(J1-Pin_13)")
-	)
-	(segment
-		(start 126.895 94.275)
-		(end 125.825 95.345)
-		(width 0.2)
-		(layer "F.Cu")
-		(net "Net-(J1-Pin_13)")
-	)
-	(segment
-		(start 115 90)
-		(end 120 95)
-		(width 0.2)
-		(layer "F.Cu")
-		(net "Net-(J1-Pin_13)")
-	)
-	(segment
-		(start 138.25 90)
-		(end 133.975 94.275)
-		(width 0.2)
-		(layer "F.Cu")
-		(net "Net-(J1-Pin_13)")
-	)
-	(segment
-		(start 120.083719 95)
-		(end 120.427091 95.343372)
-		(width 0.2)
-		(layer "F.Cu")
-		(net "Net-(J1-Pin_13)")
-	)
-	(segment
-		(start 133.975 94.275)
-		(end 126.895 94.275)
-		(width 0.2)
-		(layer "F.Cu")
-		(net "Net-(J1-Pin_13)")
-	)
-	(segment
-		(start 113.775 82.15)
-		(end 115.05 83.425)
-		(width 0.2)
-		(layer "F.Cu")
-		(net "Net-(J1-Pin_13)")
-	)
-	(segment
-		(start 113.775 81.55)
-		(end 113.775 82.15)
-		(width 0.2)
-		(layer "F.Cu")
-		(net "Net-(J1-Pin_13)")
-	)
-	(via
-		(at 120.427091 95.343372)
-		(size 0.6)
-		(drill 0.3)
-		(layers "F.Cu" "B.Cu")
-		(net "Net-(J1-Pin_13)")
-	)
-	(via
-		(at 113.775 81.55)
-		(size 0.6)
-		(drill 0.3)
-		(layers "F.Cu" "B.Cu")
-		(net "Net-(J1-Pin_13)")
-	)
-	(via
-		(at 115.05 83.425)
-		(size 0.6)
-		(drill 0.3)
-		(layers "F.Cu" "B.Cu")
-		(net "Net-(J1-Pin_13)")
-	)
-	(segment
-		(start 125.825 95.345)
-		(end 124.855 95.345)
-		(width 0.2)
-		(layer "B.Cu")
-		(net "Net-(J1-Pin_13)")
-	)
-	(segment
-		(start 123.283372 95.343372)
-		(end 124.07 96.13)
-		(width 0.2)
-		(layer "B.Cu")
-		(net "Net-(J1-Pin_13)")
-	)
-	(segment
-		(start 111.95 78.175)
-		(end 111.95 79.725)
-		(width 0.2)
-		(layer "B.Cu")
-		(net "Net-(J1-Pin_13)")
-	)
-	(segment
-		(start 115 75.125)
-		(end 111.95 78.175)
-		(width 0.2)
-		(layer "B.Cu")
-		(net "Net-(J1-Pin_13)")
-	)
-	(segment
-		(start 124.07 96.13)
-		(end 125.825 97.885)
-		(width 0.2)
-		(layer "B.Cu")
-		(net "Net-(J1-Pin_13)")
-	)
-	(segment
-		(start 125.825 115.825)
-		(end 125.825 97.885)
-		(width 0.2)
-		(layer "B.Cu")
-		(net "Net-(J1-Pin_13)")
-	)
-	(segment
-		(start 115.05 83.425)
-		(end 115 83.475)
-		(width 0.2)
-		(layer "B.Cu")
-		(net "Net-(J1-Pin_13)")
-	)
-	(segment
-		(start 115 111.5)
-		(end 119.45 115.95)
-		(width 0.2)
-		(layer "B.Cu")
-		(net "Net-(J1-Pin_13)")
-	)
-	(segment
-		(start 111.95 79.725)
-		(end 113.775 81.55)
-		(width 0.2)
-		(layer "B.Cu")
-		(net "Net-(J1-Pin_13)")
-	)
-	(segment
-		(start 120.427091 95.343372)
-		(end 123.283372 95.343372)
-		(width 0.2)
-		(layer "B.Cu")
-		(net "Net-(J1-Pin_13)")
-	)
-	(segment
-		(start 115 47)
-		(end 115 68.5)
-		(width 0.2)
-		(layer "B.Cu")
-		(net "Net-(J1-Pin_13)")
-	)
-	(segment
-		(start 115 68.5)
-		(end 115 75.125)
-		(width 0.2)
-		(layer "B.Cu")
-		(net "Net-(J1-Pin_13)")
-	)
-	(segment
-		(start 115 133)
-		(end 115 111.5)
-		(width 0.2)
-		(layer "B.Cu")
-		(net "Net-(J1-Pin_13)")
-	)
-	(segment
-		(start 119.45 115.95)
-		(end 125.95 115.95)
-		(width 0.2)
-		(layer "B.Cu")
-		(net "Net-(J1-Pin_13)")
-	)
-	(segment
-		(start 124.855 95.345)
-		(end 124.07 96.13)
-		(width 0.2)
-		(layer "B.Cu")
-		(net "Net-(J1-Pin_13)")
-	)
-	(segment
-		(start 125.95 115.95)
-		(end 125.825 115.825)
-		(width 0.2)
-		(layer "B.Cu")
-		(net "Net-(J1-Pin_13)")
-	)
-	(segment
-		(start 115 83.475)
-		(end 115 90)
-		(width 0.2)
-		(layer "B.Cu")
-		(net "Net-(J1-Pin_13)")
-	)
 	(zone

Commit message: Publish Rotary Encoder PCB version 1.3 with minor PCB changes
Other:
- board text added: "ARC-210 Rotary Encoder v1.3"
- board text removed: "ARC-210 Rotary Encoder v1.1"
Changed lines of the file:
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@@
 		)
 		(embedded_fonts no)
-		(model "PEC11H-4220F-S0024.stp"
+		(model "${KIPRJMOD}/PEC11H-4220F-S0024.stp"
 			(offset
 				(xyz 2.499999962 7.489999659 2.229999986)
@@
 		)
 		(embedded_fonts no)
-		(model "PEC11H-4220F-S0024.stp"
+		(model "${KIPRJMOD}/PEC11H-4220F-S0024.stp"
 			(offset
 				(xyz 2.499999962 7.489999659 2.229999986)
@@
 		)
 		(embedded_fonts no)
-		(model "PEC11H-4220F-S0024.stp"
+		(model "${KIPRJMOD}/PEC11H-4220F-S0024.stp"
 			(offset
 				(xyz 2.499999962 7.489999659 2.229999986)
@@
 		)
 		(embedded_fonts no)
-		(model "PEC11H-4220F-S0024.stp"
+		(model "${KIPRJMOD}/PEC11H-4220F-S0024.stp"
 			(offset
 				(xyz 2.499999962 7.489999659 2.229999986)
@@
 		)
 		(embedded_fonts no)
-		(model "PEC11H-4220F-S0024.stp"
+		(model "${KIPRJMOD}/PEC11H-4220F-S0024.stp"
 			(offset
 				(xyz 2.499999962 7.489999659 2.229999986)
@@
 		)
 	)
-	(gr_text "ARC-210 Rotary Encoder v1.1"
+	(gr_text "ARC-210 Rotary Encoder v1.3"
 		(at 105.6 89.3 90)
 		(layer "B.SilkS")

Commit message: Publish rotary encoder PCB version 1.4
Routing:
- net Net-(J1-Pin_1): track 0.00 -> 26.9 mm
- net Net-(J1-Pin_13): track 128.8 -> 127.0 mm
Other:
- board size 45.7 x 108.8 mm -> 44 x 108.8 mm
- board text added: "ARC-210 Rotary Encoder v1.4"
- board text removed: "ARC-210 Rotary Encoder v1.3"
Changed lines of the file:
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@@
 			(at 0 2.38 0)
 			(layer "B.SilkS")
+			(hide yes)
 			(effects
 				(font
@@
 			(at 0 -35.4 0)
 			(layer "B.Fab")
+			(hide yes)
 			(effects
 				(font
@@
 	)
 	(gr_line
-		(start 125.825 47.375)
-		(end 117.6 47.375)
-		(stroke
-			(width 0.2)
-			(type default)
-		)
-		(layer "F.Cu")
-		(net "Net-(J1-Pin_1)")
-	)
-	(gr_line
-		(start 125.825 64.865)
-		(end 125.825 47.375)
-		(stroke
-			(width 0.2)
-			(type default)
-		)
-		(layer "F.Cu")
-		(net "Net-(J1-Pin_1)")
-	)
-	(gr_line
 		(start 122.425 93.125)
 		(end 122.5 85.85)
@@
 	(gr_line
 		(start 102.875 28.175)
-		(end 127.600202 28.175)
-		(stroke
-			(width 0.05)
-			(type solid)
-		)
-		(layer "Edge.Cuts")
-	)
-	(gr_line
-		(start 127.55 70.15)
-		(end 148.525 70.15)
-		(stroke
-			(width 0.05)
-			(type default)
-		)
-		(layer "Edge.Cuts")
-	)
-	(gr_line
-		(start 127.575 94.875)
-		(end 127.675 137)
-		(stroke
-			(width 0.05)
-			(type default)
-		)
-		(layer "Edge.Cuts")
-	)
-	(gr_line
-		(start 127.575 94.875)
-		(end 148.55 94.875)
-		(stroke
-			(width 0.05)
-			(type default)
-		)
-		(layer "Edge.Cuts")
-	)
-	(gr_line
-		(start 127.600202 28.175)
-		(end 127.55 70.15)
-		(stroke
-			(width 0.05)
-			(type default)
-		)
-		(layer "Edge.Cuts")
-	)
-	(gr_line
-		(start 127.675 137)
-		(end 102.875 137)
-		(stroke
-			(width 0.05)
-			(type default)
-		)
-		(layer "Edge.Cuts")
-	)
-	(gr_line
-		(start 148.55 94.875)
-		(end 148.525 70.15)
+		(end 124 28.175)
+		(stroke
+			(width 0.05)
+			(type default)
+		)
+		(layer "Edge.Cuts")
+	)
+	(gr_line
+		(start 102.875 137)
+		(end 124 137)
+		(stroke
+			(width 0.05)
+			(type default)
+		)
+		(layer "Edge.Cuts")
+	)
+	(gr_line
+		(start 124 28.175)
+		(end 124 60.653368)
+		(stroke
+			(width 0.05)
+			(type default)
+		)
+		(layer "Edge.Cuts")
+	)
+	(gr_line
+		(start 124 137)
+		(end 123.975177 101.999886)
+		(stroke
+			(width 0.05)
+			(type default)
+		)
+		(layer "Edge.Cuts")
+	)
+	(gr_line
+		(start 127.3 101.05)
+		(end 123.975177 101.999886)
+		(stroke
+			(width 0.05)
+			(type default)
+		)
+		(layer "Edge.Cuts")
+	)
+	(gr_line
+		(start 127.45 62)
+		(end 124 60.653368)
+		(stroke
+			(width 0.05)
+			(type default)
+		)
+		(layer "Edge.Cuts")
+	)
+	(gr_line
+		(start 129.575 73.625)
+		(end 127.45 62)
+		(stroke
+			(width 0.05)
+			(type default)
+		)
+		(layer "Edge.Cuts")
+	)
+	(gr_line
+		(start 129.575 73.625)
+		(end 146.85 73.625)
+		(stroke
+			(width 0.05)
+			(type default)
+		)
+		(layer "Edge.Cuts")
+	)
+	(gr_line
+		(start 129.6 91.85)
+		(end 127.3 101.05)
+		(stroke
+			(width 0.05)
+			(type default)
+		)
+		(layer "Edge.Cuts")
+	)
+	(gr_line
+		(start 129.6 91.85)
+		(end 146.912917 91.85)
+		(stroke
+			(width 0.05)
+			(type default)
+		)
+		(layer "Edge.Cuts")
+	)
+	(gr_line
+		(start 146.912917 91.85)
+		(end 146.85 73.625)
 		(stroke
 			(width 0.05)
@@
 		)
 	)
-	(gr_text "ARC-210 Rotary Encoder v1.3"
+	(gr_text "ARC-210 Rotary Encoder v1.4\n"
 		(at 105.6 89.3 90)
 		(layer "B.SilkS")
@@
 	)
 	(segment
-		(start 126.895 94.275)
-		(end 125.825 95.345)
-		(width 0.2)
-		(layer "F.Cu")
-		(net "Net-(J1-Pin_13)")
-	)
-	(segment
 		(start 115 90)
 		(end 120 95)
@@
 	)
 	(segment
-		(start 138.25 90)
-		(end 133.975 94.275)
-		(width 0.2)
-		(layer "F.Cu")
-		(net "Net-(J1-Pin_13)")
-	)
-	(segment
 		(start 120.083719 95)
 		(end 120.427091 95.343372)
-		(width 0.2)
-		(layer "F.Cu")
-		(net "Net-(J1-Pin_13)")
-	)
-	(segment
-		(start 133.975 94.275)
-		(end 126.895 94.275)
 		(width 0.2)
 		(layer "F.Cu")
@@
 	)
 	(segment
+		(start 138.25 88.5)
+		(end 137.2 87.45)
+		(width 0.2)
+		(layer "B.Cu")
+		(net "Net-(J1-Pin_13)")
+	)
+	(segment
 		(start 125.825 95.345)
 		(end 124.855 95.345)
@@
 	)
 	(segment
+		(start 127.755 95.345)
+		(end 125.825 95.345)
+		(width 0.2)
+		(layer "B.Cu")
+		(net "Net-(J1-Pin_13)")
+	)
+	(segment
 		(start 123.283372 95.343372)
 		(end 124.07 96.13)
@@
 	)
 	(segment
+		(start 127.925 89.625)
+		(end 127.925 95.175)
+		(width 0.2)
+		(layer "B.Cu")
+		(net "Net-(J1-Pin_13)")
+	)
+	(segment
+		(start 125.825 97.885)
+		(end 123.21 100.5)
+		(width 0.2)
+		(layer "B.Cu")
+		(net "Net-(J1-Pin_13)")
+	)
+	(segment
+		(start 127.925 95.175)
+		(end 127.755 95.345)
+		(width 0.2)
+		(layer "B.Cu")
+		(net "Net-(J1-Pin_13)")
+	)
+	(segment
+		(start 138.25 90)
+		(end 138.25 88.5)
+		(width 0.2)
+		(layer "B.Cu")
+		(net "Net-(J1-Pin_13)")
+	)
+	(segment
 		(start 115 75.125)
 		(end 111.95 78.175)
@@
 	)
 	(segment
-		(start 125.825 115.825)
-		(end 125.825 97.885)
-		(width 0.2)
-		(layer "B.Cu")
-		(net "Net-(J1-Pin_13)")
-	)
-	(segment
 		(start 115.05 83.425)
 		(end 115 83.475)
@@
 	)
 	(segment
-		(start 115 111.5)
-		(end 119.45 115.95)
+		(start 137.2 87.45)
+		(end 130.1 87.45)
 		(width 0.2)
 		(layer "B.Cu")
@@
 	)
 	(segment
+		(start 123.21 100.5)
+		(end 115 100.5)
+		(width 0.2)
+		(layer "B.Cu")
+		(net "Net-(J1-Pin_13)")
+	)
+	(segment
 		(start 115 47)
 		(end 115 68.5)
@@
 	)
 	(segment
-		(start 119.45 115.95)
-		(end 125.95 115.95)
+		(start 130.1 87.45)
+		(end 127.925 89.625)
 		(width 0.2)
 		(layer "B.Cu")
@@
 	)
 	(segment
-		(start 125.95 115.95)
-		(end 125.825 115.825)
+		(start 115 100.5)
+		(end 115 111.5)
 		(width 0.2)
 		(layer "B.Cu")
@@
 	)
 	(segment
+		(start 119.865 64.865)
+		(end 115 60)
+		(width 0.2)
+		(layer "F.Cu")
+		(net "Net-(J1-Pin_1)")
+	)
+	(segment
+		(start 115 60)
+		(end 115 49.5)
+		(width 0.2)
+		(layer "F.Cu")
+		(net "Net-(J1-Pin_1)")
+	)
+	(segment
+		(start 125.825 64.865)
+		(end 119.865 64.865)
+		(width 0.2)
+		(layer "F.Cu")
+		(net "Net-(J1-Pin_1)")
+	)
+	(segment
+		(start 115 49.5)
+		(end 117.5 47)
+		(width 0.2)
+		(layer "F.Cu")
+		(net "Net-(J1-Pin_1)")
+	)
+	(segment
