File: PCBs/Master Board/ARC-210_Master_Board.kicad_pcb (KiCad board)
At the start: 2 copper layers, 132 x 129.2 mm, 19 parts, among them J1 SPI Display, J10 Conn_01x03_Pin, J2 4x4 Matrix, J4 Conn_01x14_Pin, J9 Conn_01x03_Pin, U1 Teensy4.1

Commit message: Remove Main Board C5/C6 to match tested direct TFT wiring; retain C1/C2 and update BOM/docs
Parts:
- removed C5: 470uF 10V, Capacitor_THT:CP_Radial_D8.0mm_P3.50mm
- removed C6: 0.1uF, Capacitor_THT:C_Disc_D5.0mm_W2.5mm_P5.00mm
- moved J1 293.2 mm to (116.3, 55.2)
- moved J4 168.0 mm to (81.3, 147.4), turned to 0 degrees
- moved U1 127.9 mm to (135.8, 116.3), turned to 90 degrees
- moved C1 124.9 mm to (116.0, 84.3), turned to -90 degrees
- moved R1 105.7 mm to (188.2, 94.9)
- moved J2 105.7 mm to (167.4, 141.3), turned to 0 degrees
- moved C2 97.8 mm to (167.2, 87.3)

Commit message: Include Teensy 4.1 STEP model and project-relative U1 attachment with 3D Viewer instructions
Parts:
- moved TP2 234.0 mm to (158.0, 74.7)
- moved TP1 217.4 mm to (149.1, 69.2)
- moved J10 162.9 mm to (185.1, 127.5)
- moved J9 156.9 mm to (152.3, 146.8)
- moved SQL1 153.9 mm to (183.5, 83.2)
- moved R2 144.1 mm to (174.0, 110.8)
Changed lines of the file:
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@@
 	(footprint "Connector_PinHeader_2.54mm:PinHeader_1x03_P2.54mm_Vertical"
 		(layer "B.Cu")
-		(at 289.356049 223.22825 180)
+		(at 152.325 146.85 180)
 		(descr "Through hole straight pin header, 1x03, 2.54mm pitch, single row")
 		(tags "Through hole pin header THT 1x03 2.54mm single row")
@@
 	(footprint "Resistor_THT:R_Axial_DIN0204_L3.6mm_D1.6mm_P5.08mm_Horizontal"
 		(layer "B.Cu")
-		(at 315.15643 82.00475 180)
+		(at 173.965 110.8 180)
 		(descr "Resistor, Axial_DIN0204 series, Axial, Horizontal, pin pitch=5.08mm, 0.167W, length*diameter=3.6*1.6mm^2, http://cdn-reichelt.de/documents/datenblatt/B400/1_4W%23YAG.pdf")
 		(tags "Resistor Axial_DIN0204 series Axial Horizontal pin pitch 5.08mm 0.167W length 3.6mm diameter 1.6mm")
@@
 	(footprint "Connector_PinHeader_2.54mm:PinHeader_1x03_P2.54mm_Vertical"
 		(layer "B.Cu")
-		(at 316.844145 223.22825 180)
+		(at 185.075 127.475 180)
 		(descr "Through hole straight pin header, 1x03, 2.54mm pitch, single row")
 		(tags "Through hole pin header THT 1x03 2.54mm single row")
@@
 		)
 		(embedded_fonts no)
-		(model "${KICAD_USER_DIR}/teensy.pretty/Teensy_4.1_Assembly.STEP"
+		(model "${KIPRJMOD}/Libraries/3dmodels/Teensy_4.1_Board.step"
 			(offset
 				(xyz 0 0 0.762)
@@
 	(footprint "TestPoint:TestPoint_THTPad_D3.0mm_Drill1.5mm"
 		(layer "B.Cu")
-		(at 391.923098 82.48475 180)
+		(at 158.025 74.675 180)
 		(descr "THT pad as test Point, diameter 3.0mm, hole diameter 1.5mm")
 		(tags "test point THT pad")
@@
 	(footprint "Connector_PinHeader_2.54mm:PinHeader_1x02_P2.54mm_Vertical"
 		(layer "B.Cu")
-		(at 337.375478 82.46475 180)
+		(at 183.525 83.225 180)
 		(descr "Through hole straight pin header, 1x02, 2.54mm pitch, single row")
 		(tags "Through hole pin header THT 1x02 2.54mm single row")
@@
 	(footprint "TestPoint:TestPoint_THTPad_D3.0mm_Drill1.5mm"
 		(layer "B.Cu")
-		(at 366.05405 82.48475 180)
+		(at 149.075 69.2 180)
 		(descr "THT pad as test Point, diameter 3.0mm, hole diameter 1.5mm")
 		(tags "test point THT pad")

Commit message: Publish current Main Board layout and schematic with check reports
Parts:
- J10: value Conn_01x03_Pin -> MASTER
- J4: value Conn_01x14_Pin -> ROTARY ENCODERS
- J9: value Conn_01x03_Pin -> MODE
- TP1: value SQL_ONOFF_GPIO41 -> SQL ON/OFF
- moved J2 75.4 mm to (134.2, 73.6), turned to 90 degrees
- moved SQL1 54.0 mm to (137.9, 54.2)
- moved C1 46.8 mm to (153.7, 112.0), turned to 180 degrees
- moved C2 34.3 mm to (151.2, 117.7), turned to 0 degrees
- moved R1 32.6 mm to (160.3, 111.9), turned to 0 degrees
- moved J1 29.0 mm to (87.4, 52.9), turned to -90 degrees
- moved J10 24.7 mm to (169.8, 146.9)
- moved TP1 18.5 mm to (149.1, 50.7)
- moved TP2 15.2 mm to (149.1, 62.4)
- moved R2 11.1 mm to (165.4, 117.9)
Connections:
- U1 pad 64: GND -> unconnected-(U1-GND-Pad64)
Routing:
- net GND: track 0.00 -> 410.5 mm, vias 0 -> 2
- net /TEENSY_3V3: track 0.00 -> 159.8 mm, vias 0 -> 2
- net /ENC3_B: track 0.00 -> 140.2 mm, vias 0 -> 2
- net /TFT_SCK: track 0.00 -> 128.7 mm
- net /ENC3_A: track 0.00 -> 118.6 mm
- net /ENC1_B: track 0.00 -> 116.8 mm
- net /ENC2_A: track 0.00 -> 110.4 mm, vias 0 -> 3
- net /ENC2_B: track 0.00 -> 110.3 mm
- net /ENC1_A: track 0.00 -> 110.2 mm, vias 0 -> 2
- net /ENC4_A: track 0.00 -> 107.0 mm
- net Net-(J1-Pin_3): track 0.00 -> 101.6 mm, vias 0 -> 3
- net /TFT_CS: track 0.00 -> 94.9 mm, vias 0 -> 2
- net Net-(J1-Pin_8): track 0.00 -> 93.8 mm
- net /ENC4_B: track 0.00 -> 93.0 mm
- net Net-(J1-Pin_6): track 0.00 -> 88.5 mm, vias 0 -> 2
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Other:
- board text added: "INSTALL COMPONENTS ON THE OTHER SIDE"
- board text added: "INSTALL COMPONENTS ON THIS SIDE"
- board text removed: "COMPONENTS ON BACK AWAY FROM FACEPLATE"
