File: PCBs/Master Board/ARC-210_Master_Board.kicad_pcb (KiCad board)
At the start: 2 copper layers, 132 x 129.2 mm, 17 parts, among them J1 SPI Display, J10 MASTER, J2 4x4 Matrix, J4 ROTARY ENCODERS, J9 MODE, U1 Teensy4.1

Commit message: Publish Main Board v1.1 ground pours and refresh build documentation
Routing:
- added copper zone on B.Cu, net GND
- added copper zone on F.Cu, net GND
Other:
- board text added: "ARC-210 https://github.com/dgdimick/ARC-210-DCS-Display Main Controler Board v1.1"
- board text removed: "ARC-210 https://github.com/dgdimick/ARC-210-DCS-Display Main Controler Board v1.0"
Changed lines of the file:
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@@
 	)
 	(paper "A4")
+	(title_block
+		(rev "1.1")
+	)
 	(layers
 		(0 "F.Cu" signal)
@@
 		(layer "Edge.Cuts")
 	)
+	(gr_line
+		(start 127.21 162.5)
+		(end 127.21 164.5)
+		(stroke
+			(width 0.05)
+			(type default)
+		)
+		(layer "Edge.Cuts")
+	)
+	(gr_arc
+		(start 127.21 162.5)
+		(mid 128.21 161.5)
+		(end 129.21 162.5)
+		(stroke
+			(width 0.05)
+			(type default)
+		)
+		(layer "Edge.Cuts")
+	)
+	(gr_arc
+		(start 129.21 164.5)
+		(mid 128.21 165.5)
+		(end 127.21 164.5)
+		(stroke
+			(width 0.05)
+			(type default)
+		)
+		(layer "Edge.Cuts")
+	)
+	(gr_line
+		(start 129.21 164.5)
+		(end 129.21 162.5)
+		(stroke
+			(width 0.05)
+			(type default)
+		)
+		(layer "Edge.Cuts")
+	)
+	(gr_line
+		(start 142.45 162.5)
+		(end 142.45 164.5)
+		(stroke
+			(width 0.05)
+			(type default)
+		)
+		(layer "Edge.Cuts")
+	)
+	(gr_arc
+		(start 142.45 162.5)
+		(mid 143.45 161.5)
+		(end 144.45 162.5)
+		(stroke
+			(width 0.05)
+			(type default)
+		)
+		(layer "Edge.Cuts")
+	)
+	(gr_arc
+		(start 144.45 164.5)
+		(mid 143.45 165.5)
+		(end 142.45 164.5)
+		(stroke
+			(width 0.05)
+			(type default)
+		)
+		(layer "Edge.Cuts")
+	)
+	(gr_line
+		(start 144.45 164.5)
+		(end 144.45 162.5)
+		(stroke
+			(width 0.05)
+			(type default)
+		)
+		(layer "Edge.Cuts")
+	)
 	(gr_arc
 		(start 164.125 70.625)
@@
 		)
 	)
-	(gr_text "ARC-210 https://github.com/dgdimick/ARC-210-DCS-Display\nMain Controler Board v1.0\n"
+	(gr_text "ARC-210 https://github.com/dgdimick/ARC-210-DCS-Display\nMain Controler Board v1.1\n"
 		(at 191.86 69.42 90)
 		(layer "B.SilkS")
@@
 		(net "/TFT_SCK")
 	)
+	(zone
+		(net "GND")
+		(layers "F.Cu" "B.Cu")
+		(hatch edge 0.5)
+		(connect_pads
+			(clearance 0.5)
+		)
+		(min_thickness 0.25)
+		(fill yes
+			(thermal_gap 0.5)
+			(thermal_bridge_width 0.5)
+			(island_removal_mode 0)
+		)
+		(polygon
+			(pts
+				(xy 52.64 33.49) (xy 56.09 179.07) (xy 222.06 178.5) (xy 213.44 27.75) (xy 52.67 33.52)
+			)
+		)
+	)
 	(embedded_fonts no)
-(gr_line (start 127.21000000000001 162.5) (end 127.21000000000001 164.5) (stroke (width 0.05) (type default)) (layer "Edge.Cuts"))
-(gr_arc (start 127.21000000000001 164.5) (mid 128.21 165.5) (end 129.21 164.5) (stroke (width 0.05) (type default)) (layer "Edge.Cuts"))
-(gr_line (start 129.21 164.5) (end 129.21 162.5) (stroke (width 0.05) (type default)) (layer "Edge.Cuts"))
-(gr_arc (start 129.21 162.5) (mid 128.21 161.5) (end 127.21000000000001 162.5) (stroke (width 0.05) (type default)) (layer "Edge.Cuts"))
-(gr_line (start 142.45 162.5) (end 142.45 164.5) (stroke (width 0.05) (type default)) (layer "Edge.Cuts"))
-(gr_arc (start 142.45 164.5) (mid 143.45 165.5) (end 144.45 164.5) (stroke (width 0.05) (type default)) (layer "Edge.Cuts"))
-(gr_line (start 144.45 164.5) (end 144.45 162.5) (stroke (width 0.05) (type default)) (layer "Edge.Cuts"))
-(gr_arc (start 144.45 162.5) (mid 143.45 161.5) (end 142.45 162.5) (stroke (width 0.05) (type default)) (layer "Edge.Cuts"))
 )
