File: PCBs/Master Board/ARC-210_Master_Board.kicad_sch (KiCad schematic)
At the start: 23 parts, among them J1 SPI Display, J10 Conn_01x03_Pin, J2 4x4 Matrix, J3 5.0V-5.5V INPUT, J4 Conn_01x14_Pin, J9 Conn_01x03_Pin, Q2 C106D SCR, U1 Teensy4.1

Commit message: Publish USB-powered Main Board draft with direct 3.3V TFT supply and updated build documentation
Parts:
- removed D1: SB560, Diode_THT:D_DO-201AD_P15.24mm_Horizontal, symbol Device:D_Schottky
- removed D2: POWER GREEN, LED_THT:LED_D5.0mm, symbol Device:LED
- removed D3: 1N4734A 5.6V, Diode_THT:D_DO-41_SOD81_P10.16mm_Horizontal, symbol Device:D_Zener
- removed F2: 1.1A HOLD PTC, symbol Device:Polyfuse
- removed J3: 5.0V-5.5V INPUT, symbol Connector:Barrel_Jack
- removed JP1: TFT_POWER_SELECT, Connector_PinHeader_2.54mm:PinHeader_1x03_P2.54mm_Vertical, symbol Jumper:Jumper_3_Open
- removed Q2: C106D SCR, symbol ARC210_Power:C106D
- removed R15, R17: 1k, symbol Device:R
- removed R16: 220, symbol Device:R
- added TP1: SQL_ONOFF_GPIO41, TestPoint:TestPoint_THTPad_D3.0mm_Drill1.5mm, symbol Connector:TestPoint
- added TP2: SQL_GND, TestPoint:TestPoint_THTPad_D3.0mm_Drill1.5mm, symbol Connector:TestPoint
- J10, J9: footprint (none) -> Connector_PinHeader_2.54mm:PinHeader_1x03_P2.54mm_Vertical
- J2: footprint (none) -> Connector_PinHeader_2.54mm:PinHeader_1x08_P2.54mm_Vertical
Connections:
- net PANEL_5V is gone; now on net TEENSY_3V3: C5.1, C6.1
- net TFT_VCC is gone; now on net TEENSY_3V3: J1.1 (Pin_1)
- net GND: now also TP2.1
- net SQL_ONOFF: now reaches SQL1.1 (Pin_1), U1.33 (41_A17)
- net SQL_ONOFF: now also TP1.1
Other:
- note added: "3.3 VOLTS"
- note added: "SQL On/Off direct solder-wire option TP1: GPIO 41 (U1 pad 33); TP2: GND Solder-lug switch: common to TP1, selected contact to TP2 Configure GPIO 41 with a pull-up. SQL1 header remains optional."
- note added: "USB-powered Main Board: TFT VCC connects directly to TEENSY_3V3 (U1 pad 15). External protected 5V input and JP1 removed. C5/C6 retained as 3.3V decoupling. TFT brightness at 3.3V confirmed satisfactory. Total external 3.3V load: 250 mA maximum recommended."
- note removed: "5 VOLTS"
- note removed: "At 5.5V input, D1 normally puts PANEL_5V near 5.0-5.3V. Verify J2 voltage before connecting the TFT."
- note removed: "Connect Teensy pin 39 and one Teensy GND pin only. Never connect PANEL_5V to Teensy VIN or 3.3V."
- note removed: "EXTERNAL POWER INPUT AND PROTECTION"
- note removed: "Expected ARC-210 load: 16 LEDs about 0.20-0.25A plus TFT. The 1.1A PTC allows operating and startup margin."
- note removed: "Power future ARC-186/KY-58 panels from separately fused branches rather than through this ARC-210 branch."
- note removed: "Protection/filtering for a regulated 5.0V-5.5V adapter; this is not a precision 5V regulator."
- note removed: "TFT power: fit jumper 1-2 for protected 5V OR 2-3 for Teensy 3.3V. Fit ONE jumper shunt only. Remove power before changing. Default: no shunt. 3.3V option: verify total external load stays within 250mA."
- note removed: "Use 1/2 Watt Resistors"

Commit message: Remove Main Board C5/C6 to match tested direct TFT wiring; retain C1/C2 and update BOM/docs
Parts:
- removed C5: 470uF 10V, Capacitor_THT:CP_Radial_D8.0mm_P3.50mm, symbol Device:C_Polarized
- removed C6: 0.1uF, Capacitor_THT:C_Disc_D5.0mm_W2.5mm_P5.00mm, symbol Device:C
Other:
- note added: "USB-powered Main Board: TFT VCC connects directly to TEENSY_3V3 (U1 pad 15). External protected 5V input and JP1 removed. C5/C6 removed to match the tested direct TFT wiring. C1/C2 rotary filters retained. TFT brightness at 3.3V confirmed satisfactory. Total external 3.3V load: 250 mA maximum recommended."
- note removed: "USB-powered Main Board: TFT VCC connects directly to TEENSY_3V3 (U1 pad 15). External protected 5V input and JP1 removed. C5/C6 retained as 3.3V decoupling. TFT brightness at 3.3V confirmed satisfactory. Total external 3.3V load: 250 mA maximum recommended."
Changed lines of the file:
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@@
-	)
-	(symbol
-		(lib_id "Device:C")
-		(at 204.47 312.42 0)
-		(unit 1)
-		(body_style 1)
-		(exclude_from_sim no)
-		(in_bom yes)
-		(on_board yes)
-		(in_pos_files yes)
-		(dnp no)
-		(property "Reference" "C6"
-			(at 200.66 309.88 0)
-			(show_name no)
-			(do_not_autoplace no)
-			(effects
-				(font
-					(size 1.27 1.27)
-				)
-			)
-		)
-		(property "Value" "0.1uF"
-			(at 209.55 312.42 90)
-			(show_name no)
-			(do_not_autoplace no)
-			(effects
-				(font
-					(size 1.27 1.27)
-				)
-			)
-		)
-		(property "Footprint" "Capacitor_THT:C_Disc_D5.0mm_W2.5mm_P5.00mm"
-			(at 204.47 312.42 0)
-			(hide yes)
-			(show_name no)
-			(do_not_autoplace no)
-			(effects
-				(font
-					(size 1.27 1.27)
-				)
-			)
-		)
-		(property "Datasheet" ""
-			(at 204.47 312.42 0)
-			(show_name no)
-			(do_not_autoplace no)
-			(effects
-				(font
-					(size 1.27 1.27)
-				)
-			)
-		)
-		(property "Description" "Unpolarized capacitor"
-			(at 209.55 312.42 90)
-			(hide yes)
-			(show_name no)
-			(do_not_autoplace no)
-			(effects
-				(font
-					(size 1.27 1.27)
-				)
-			)
-		)
-		(pin "2"
-		)
-		(pin "1"
-		)
-		(instances
-			(project "ARC-210_Master_Board"
-				(path "/0e535162-9d69-490e-913e-7ee098d37ead"
-					(reference "C6")
-					(unit 1)
-				)
-			)
-		)
 	)
 	(symbol
@@
 				(path "/0e535162-9d69-490e-913e-7ee098d37ead"
 					(reference "#FLG01")
-					(unit 1)
-				)
-			)
-		)
-	)
-	(symbol
-		(lib_id "Device:C_Polarized")
-		(at 186.69 312.42 0)
-		(unit 1)
-		(body_style 1)
-		(exclude_from_sim no)
-		(in_bom yes)
-		(on_board yes)
-		(in_pos_files yes)
-		(dnp no)
-		(property "Reference" "C5"
-			(at 190.5 309.88 0)
-			(show_name no)
-			(do_not_autoplace no)
-			(effects
-				(font
-					(size 1.27 1.27)
-				)
-			)
-		)
-		(property "Value" "470uF 10V"
-			(at 182.88 312.42 90)
-			(show_name no)
-			(do_not_autoplace no)
-			(effects
-				(font
-					(size 1.27 1.27)
-				)
-			)
-		)
-		(property "Footprint" "Capacitor_THT:CP_Radial_D8.0mm_P3.50mm"
-			(at 186.69 312.42 0)
-			(hide yes)
-			(show_name no)
-			(do_not_autoplace no)
-			(effects
-				(font
-					(size 1.27 1.27)
-				)
-			)
-		)
-		(property "Datasheet" ""
-			(at 186.69 312.42 0)
-			(show_name no)
-			(do_not_autoplace no)
-			(effects
-				(font
-					(size 1.27 1.27)
-				)
-			)
-		)
-		(property "Description" "Polarized capacitor"
-			(at 181.61 313.69 90)
-			(hide yes)
-			(show_name no)
-			(do_not_autoplace no)
-			(effects
-				(font
-					(size 1.27 1.27)
-				)
-			)
-		)
-		(pin "2"
-		)
-		(pin "1"
-		)
-		(instances
-			(project "ARC-210_Master_Board"
-				(path "/0e535162-9d69-490e-913e-7ee098d37ead"
-					(reference "C5")
 					(unit 1)
 				)
@@
         (pin "1") (instances (project "ARC-210_Master_Board" (path "/0e535162-9d69-490e-913e-7ee098d37ead" (reference "#PWR0999") (unit 1)))))
 (text "SQL On/Off direct solder-wire option\nTP1: GPIO 41 (U1 pad 33); TP2: GND\nSolder-lug switch: common to TP1, selected contact to TP2\nConfigure GPIO 41 with a pull-up. SQL1 header remains optional." (at 720 235 0) (effects (font (size 1.27 1.27))))
-(label "TEENSY_3V3" (at 186.69 308.61 0) (effects (font (size 1.27 1.27)) (justify left bottom)))
-(symbol (lib_id "power:GND") (at 186.69 316.23 0) (unit 1) (in_bom yes) (on_board yes) (dnp no)
-(property "Reference" "#PWR0501" (at 186.69 316.23 0) (hide yes) (effects (font (size 1.27 1.27)))) (property "Value" "GND" (at 186.69 320.04 0) (effects (font (size 1.27 1.27)))) (pin "1")
-(instances (project "ARC-210_Master_Board" (path "/0e535162-9d69-490e-913e-7ee098d37ead" (reference "#PWR0501") (unit 1)))))
-(label "TEENSY_3V3" (at 204.47 308.61 0) (effects (font (size 1.27 1.27)) (justify left bottom)))
-(symbol (lib_id "power:GND") (at 204.47 316.23 0) (unit 1) (in_bom yes) (on_board yes) (dnp no)
-(property "Reference" "#PWR0502" (at 204.47 316.23 0) (hide yes) (effects (font (size 1.27 1.27)))) (property "Value" "GND" (at 204.47 320.04 0) (effects (font (size 1.27 1.27)))) (pin "1")
-(instances (project "ARC-210_Master_Board" (path "/0e535162-9d69-490e-913e-7ee098d37ead" (reference "#PWR0502") (unit 1)))))
 (symbol (lib_id "power:GND") (at 195.58 330.2 0) (unit 1) (in_bom yes) (on_board yes) (dnp no)
 (property "Reference" "#PWR029" (at 195.58 330.2 0) (hide yes) (effects (font (size 1.27 1.27)))) (property "Value" "GND" (at 195.58 334.01 0) (effects (font (size 1.27 1.27)))) (pin "1")
@@
 (property "Reference" "#FLG02" (at 195.58 330.2 0) (hide yes) (effects (font (size 1.27 1.27)))) (property "Value" "PWR_FLAG" (at 195.58 334.01 0) (hide yes) (effects (font (size 1.27 1.27)))) (pin "1")
 (instances (project "ARC-210_Master_Board" (path "/0e535162-9d69-490e-913e-7ee098d37ead" (reference "#FLG02") (unit 1)))))
-(text "USB-powered Main Board: TFT VCC connects directly to TEENSY_3V3 (U1 pad 15).\nExternal protected 5V input and JP1 removed. C5/C6 retained as 3.3V decoupling.\nTFT brightness at 3.3V confirmed satisfactory. Total external 3.3V load: 250 mA maximum recommended." (at 210.82 284.48 0) (effects (font (size 1.27 1.27))))
+(text "USB-powered Main Board: TFT VCC connects directly to TEENSY_3V3 (U1 pad 15).\nExternal protected 5V input and JP1 removed. C5/C6 removed to match the tested direct TFT wiring. C1/C2 rotary filters retained.\nTFT brightness at 3.3V confirmed satisfactory. Total external 3.3V load: 250 mA maximum recommended." (at 210.82 284.48 0) (effects (font (size 1.27 1.27))))
 )

Commit message: Publish current Main Board layout and schematic with check reports
Parts:
- J10: value Conn_01x03_Pin -> MASTER
- J9: value Conn_01x03_Pin -> MODE
Connections:
- net GND: no longer U1.64 (GND)
- no-connect marks 31 -> 32

Commit message: Match J4 and TP1 schematic values and update project completion list
Parts:
- J4: value Conn_01x14_Pin -> ROTARY ENCODERS
- TP1: value SQL_ONOFF_GPIO41 -> SQL ON/OFF
Changed lines of the file:
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@@
 			)
 		)
-		(property "Value" "Conn_01x14_Pin"
+		(property "Value" "ROTARY ENCODERS"
 			(at 254 374.015 0)
 			(show_name no)
@@
 			)
 		)
-		(property "Value" "SQL_ONOFF_GPIO41"
+		(property "Value" "SQL ON/OFF"
 			(at 703.5 206 0)
 			(show_name no)

Commit message: Publish Main Board v1.1 ground pours and refresh build documentation
Other:
- title: (none) -> ARC-210 Main Board
Changed lines of the file:
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@@
 	(generator_version "10.0")
 	(paper "A1")
+	(title_block (title "ARC-210 Main Board") (rev "1.1"))
 	(text "SCK"
 		(exclude_from_sim no)
