File: PCBs/Button Matrix/Button Matrix.kicad_pcb (KiCad board)
At the start: 2 copper layers, 143.5 x 129.2 mm, 39 parts, among them J1 Conn_01x04_Pin, J2 Conn_01x04_Pin, SW1 SW_Push, SW10 SW_Push, SW11 SW_Push, SW12 SW_Push, SW13 SW_Push, SW14 SW_Push, SW15 SW_Push, SW16 SW_Push, SW2 SW_Push, SW3 SW_Push, SW4 SW_Push, SW5 SW_Push, SW6 SW_Push, SW7 SW_Push, SW8 SW_Push, SW9 SW_Push

Commit message: Release Button Matrix v3.2 with fresh manufacturing exports and latest update preview
Other:
- board text added: "ARC-210 v3.2"
- board text removed: "ARC-210 v3.1"
Changed lines of the file:
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@@
 	(paper "A3")
 	(title_block
-		(rev "3.1")
+		(rev "3.2")
 	)
 	(layers
@@
 		(tags "mounting hole NPTH 12mm")
 		(property "Reference" "H3"
-			(at 0 -4.45 0)
+			(at 9 0 0)
 			(layer "F.SilkS")
 			(effects
@@
 		(layer "Edge.Cuts")
 	)
-	(gr_text "ARC-210 v3.1\n"
+	(gr_text "ARC-210 v3.2"
 		(at 179.375 155.075 0)
 		(layer "B.SilkS")
